File: fumexDriver.kicad_pcb (KiCad board)
At the start: 2 copper layers, 83.3 x 92.3 mm, 102 parts, among them J1 PWR, J2 FAN, J3 STAND, J4 68000-103HLF, K1 AZ943-1AH-12DE, Q1 BC847, Q2 2N7002, Q3 BC847, SW1 LC1258EENP, U1 NE556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

Commit message: Release 1.0.0
Parts:
- removed D10, D11: LL103A, Diode_SMD:D_MiniMELF
- added C23: 100n, Capacitor_SMD:C_0603_1608Metric, F.Cu at (171.5, 116.8)
- added C24: 100n, Capacitor_SMD:C_0603_1608Metric, F.Cu at (191.0, 120.3)
- added C25: 1u, Capacitor_SMD:C_0603_1608Metric, F.Cu at (165.1, 116.9)
- added C26: 100n, Capacitor_SMD:C_0603_1608Metric, F.Cu at (182.6, 114.8)
- added C27: 100n, Capacitor_SMD:C_0603_1608Metric, F.Cu at (176.9, 87.9)
- added NT1: NetTie_2, Resistor_SMD:R_1206_3216Metric_Pad1.30x1.75mm_HandSolder, F.Cu at (182.3, 103.2)
- added NT2: NetTie_2, Resistor_SMD:R_1206_3216Metric_Pad1.30x1.75mm_HandSolder, F.Cu at (185.6, 103.2)
- added Q4: BC847, Package_TO_SOT_SMD:SOT-23, F.Cu at (171.1, 112.5)
- added Q5: BC847, Package_TO_SOT_SMD:SOT-23, F.Cu at (171.2, 108.8)
- added R21: 3k3, Resistor_SMD:R_0603_1608Metric, F.Cu at (157.1, 111.6)
- added R22: 3k3, Resistor_SMD:R_0603_1608Metric, F.Cu at (171.5, 115.1)
- added R23: 3k3, Resistor_SMD:R_0603_1608Metric, F.Cu at (174.9, 107.8)
- added R24: 10k, Resistor_SMD:R_0603_1608Metric, F.Cu at (144.3, 117.2)
- added R25: 10k, Resistor_SMD:R_0603_1608Metric, F.Cu at (144.3, 115.4)
- added R26: 47k, Resistor_SMD:R_0603_1608Metric, F.Cu at (165.1, 115.1)
- added TP20: ~, TestPoint:TestPoint_Pad_D1.0mm, F.Cu at (175.7, 104.5)
- moved TP13 19.6 mm to (189.5, 124.0), turned to 180 degrees
- moved TP16 17.3 mm to (168.7, 120.3)
- moved TP17 17.1 mm to (175.7, 101.7)
- moved D20 15.5 mm to (165.1, 112.5), turned to 180 degrees
- moved D17 14.9 mm to (186.0, 122.2), turned to 180 degrees
- moved R7 14.1 mm to (185.6, 120.3), turned to 180 degrees
- moved D16 12.2 mm to (173.4, 122.2), turned to 0 degrees
- moved R8 11.4 mm to (173.8, 120.3), turned to 180 degrees
- moved TP19 6.77 mm to (184.2, 118.1)
- moved TP14 5.22 mm to (178.2, 117.9)
- moved D7 3.85 mm to (164.3, 108.0)
- moved R12 3.80 mm to (163.2, 105.9), turned to 0 degrees
- moved R9 3.76 mm to (163.2, 104.2), turned to 0 degrees
- moved C10 2.00 mm to (188.0, 112.0)
- moved C9 1.53 mm to (179.4, 109.7)
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Connections:
- D20 pad 2: Net-(D11-A) -> Net-(D7-K)
- D7 pad 1: Net-(D11-A) -> Net-(D7-K)
- J4 pad 2: Net-(D11-A) -> Net-(J4-Pin_2)
- RV1 pad 1: Net-(D17-A2) -> Net-(D16-A2)
- RV1 pad 3: Net-(D16-A2) -> Net-(D17-A2)
- TP16 pad 1: Net-(D11-A) -> Net-(Q4-B)
- U1 pad 3: +12VA -> Net-(U1A-CV)
- U2 pad 2: Net-(D11-A) -> Net-(Q4-B)
- U2 pad 5: unconnected-(U2-CV-Pad5) -> Net-(U2-CV)
- U3 pad 5: (no net) -> Net-(U3B-+)
- U3 pad 6: (no net) -> Net-(U3B--)
- U3 pad 7: (no net) -> unconnected-(U3-Pad7)
Routing:
- net Net-(D11-A): track 47.0 -> 0.00 mm, vias 2 -> 0
- net Net-(Q4-B): track 0.00 -> 26.1 mm
- net Net-(Q2-G): track 41.7 -> 64.0 mm
- net Net-(D7-K): track 0.00 -> 21.5 mm
- net Net-(U2-Q): track 25.0 -> 11.6 mm
- net GND: track 74.3 -> 84.4 mm, vias 53 -> 62
- net Net-(D4-A2): track 55.3 -> 60.1 mm
- net +12VA: track 32.3 -> 36.6 mm
- net Net-(Q5-B): track 0.00 -> 3.51 mm
- net Net-(U3B-+): track 0.00 -> 3.02 mm
- net Net-(U3B--): track 0.00 -> 2.97 mm
- net Net-(U2-CV): track 0.00 -> 2.42 mm
- net Net-(J4-Pin_2): track 0.00 -> 2.38 mm
- net Net-(U1A-CV): track 0.00 -> 2.03 mm
- net Net-(D17-A2): track 14.4 -> 16.0 mm
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Other:
- board text added: "Fuse 2A 5x20mm"

Commit message: Release 1.2.0
Parts:
- added R27: 3k3, Resistor_SMD:R_0603_1608Metric, F.Cu at (165.1, 118.8)
- FH1: footprint Fuse_Holders:ESKA_503.400 -> Koszalix_FuseHolders:ESKA_503.400
- K1: footprint Relays:Zettler_AZ943 -> Koszalix_Relays:Zettler_AZ943
- RV1: footprint Potentiometer:SR_PASSIVES_R16148 -> Koszalix_Poteniometer:SR_PASSIVES_R16148
- moved TP16 4.51 mm to (164.3, 121.3)
Connections:
- C25 pad 1: Net-(Q4-B) -> Net-(U2-TR)
- R26 pad 2: Net-(Q4-B) -> Net-(U2-TR)
- TP16 pad 1: Net-(Q4-B) -> Net-(U2-TR)
- U2 pad 2: Net-(Q4-B) -> Net-(U2-TR)
Routing:
- net Net-(U2-TR): track 0.00 -> 23.2 mm
- net Net-(Q4-B): track 26.1 -> 13.6 mm
Other:
- board text added: "Fumex Driver Rev 1.2.0 11/2023"
- board text removed: "Fumex Driver Rev 1.0.0 11/2023"
