File: psu.kicad_sch (KiCad schematic)
At the start: 43 parts, among them J1 PWR, K1 AZ943-1AH-12DE, Q1 BC847, SW1 LC1258EENP, U3 LM393

Commit message: Release 1.0.0
Parts:
- added NT1, NT2: NetTie_2, Resistor_SMD:R_1206_3216Metric_Pad1.30x1.75mm_HandSolder, symbol Device:NetTie_2
- added R24, R25: 10k, Resistor_SMD:R_0603_1608Metric, symbol RES_YAGEO_RC0603:RES_10k_0603
- added unit 2 of U3
Connections:
- net +12P: now also R25.1
- net +12VA: now also NT1.1, NT1.2, NT2.1, NT2.2
- net GND: now also R24.1
- new net: R24.2, U3.5 (+)
- new net: R25.2, U3.6 (-)
- no-connect marks 2 -> 3
Other:
- note added: "Jumpers"
- moved on the sheet: D15

Commit message: Release 1.2.0
Parts:
- FH1: footprint Fuse_Holders:ESKA_503.400 -> Koszalix_FuseHolders:ESKA_503.400
- K1: footprint Relays:Zettler_AZ943 -> Koszalix_Relays:Zettler_AZ943
Changed lines of the file:
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@@
       (effects (font (size 1.27 1.27)))
     )
-    (property "Footprint" "Relays:Zettler_AZ943" (at 179.705 59.69 0)
+    (property "Footprint" "Koszalix_Relays:Zettler_AZ943" (at 179.705 59.69 0)
       (effects (font (size 1.27 1.27)) (justify left) hide)
     )
@@
       (effects (font (size 1.27 1.27)) (justify left))
     )
-    (property "Footprint" "Relays:Zettler_AZ943" (at 200.66 100.965 0)
+    (property "Footprint" "Koszalix_Relays:Zettler_AZ943" (at 200.66 100.965 0)
       (effects (font (size 1.27 1.27)) (justify left) hide)
     )
@@
       (effects (font (size 1.27 1.27)))
     )
-    (property "Footprint" "Fuse_Holders:ESKA_503.400" (at 48.895 26.035 0)
-      (effects (font (size 1.27 1.27)) (justify left) hide)
-    )
+    (property "Footprint" "Koszalix_FuseHolders:ESKA_503.400" (at 48.895 26.035 0)
+      (effects (font (size 1.27 1.27)) (justify left) hide)
+    )
